File: TarjetaMod/TarjetaMod.kicad_sch (KiCad schematic)
At the start: 70 parts, among them J10 691311500008, J11 691311500018, J12 691311500002, J13 691311500018, J14 691311500002, J2 691311500008, J3 691311500018, J4 691311500016, J5 691311500006, J6 691311500004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

Commit message: Acomodo de componentes en el diagrama esquemático.
Other:
- note added: "Faltan capacitores de acople, se añaden cuando se termine la revisión."
- note removed: "Agregar los huecos para los trimmers (jumpers del micro)(LISTO) Poner en DigiKey, los conectores entre microcontrolador y tarjeta. (LISTO o CASI LISTO) Ver cómo alimentar el circuito (buscar un LDO? de 1.6 V). (LISTO) Faltan capis de acople (SE VAN AGREGANDO CONFORME HAGO LA PCB) Posiblemente hay que cambiar la configuración del circuito buffer del EN para que de 0 o 5 V. (LISTO)"
Changed lines of the file:
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@@
 	(title_block
 		(title "Tarjeta microcontrolador")
-		(date "2026-03-13")
+		(date "2026-06-28")
 		(rev "v.1")
 		(company "LabCES - UCR")
-	)
-	(text "Agregar los huecos para los trimmers (jumpers del micro)(LISTO)\nPoner en DigiKey, los conectores entre microcontrolador y tarjeta. (LISTO o CASI LISTO)\nVer cómo alimentar el circuito (buscar un LDO? de 1.6 V). (LISTO)\nFaltan capis de acople (SE VAN AGREGANDO CONFORME HAGO LA PCB)\nPosiblemente hay que cambiar la configuración del circuito buffer del EN para que de 0 o 5 V. (LISTO)"
-		(exclude_from_sim no)
-		(at 301.498 206.756 0)
-		(effects
-			(font
-				(size 1.27 1.27)
-			)
-		)
 	)
 	(text "Configuración Buffer\n"
@@
 		(exclude_from_sim no)
 		(at 109.728 127.508 0)
+		(effects
+			(font
+				(size 1.27 1.27)
+			)
+		)
+	)
+	(text "Faltan capacitores de acople,\nse añaden cuando se termine la revisión."
+		(exclude_from_sim no)
+		(at 133.096 387.096 0)
 		(effects
 			(font
@@
 	(text_box "TRACO de +15 V y - 15 V\nConvertidor DC/DC"
 		(exclude_from_sim no)
-		(at 481.965 340.995 0)
-		(size 110.49 32.385)
+		(at 360.045 180.975 0)
+		(size 118.745 175.895)
 		(margins 0.9525 0.9525 0.9525 0.9525)
 		(stroke
